File: Bucket_universel_v2_before_buck_rework.kicad_pcb (KiCad board)
At the start: 2 copper layers, 100 x 60.5 mm, 128 parts, among them J1 Conn_02x11_Odd_Even, J10 Conn_01x03, J11 Conn_01x03, J12 Conn_01x04_Pin, J13 SM03B-SRSS-TB, J14 Conn_02x18_Odd_Even, J15 USB_C_Receptacle_USB2.0_16P, J2 Conn_01x03_Pin, J3 Conn_01x05_Pin, J4 Conn_01x04_Pin, J5 Conn_01x04_Pin, J7 Conn_02x18_Odd_Even, J8 Conn_01x03, J9 Conn_01x02_Pin, SW1 SW_Push, SW2 SW_Push, U1 DRV8825PWPR, U10 SN74LVC1T45DBV, U11 DRV8874PWPR, U12 LM7805MP/NOPB, U2 DRV8874PWPR, U3 W25Q128JVS, U4 NCP1117-3.3_SOT223, U5 RP2350_60QFN, U7 SN74LVC1T45DBV, U8 AOZ2261AQI-15, U9 SN74LVC1T45DBV, Y1 ABM8-272-T3

Commit message: Yes
Parts:
- J15: footprint Rework_local:USB4105_GND_heel_relief -> Connector_USB:USB_C_Receptacle_GCT_USB4105-xx-A_16P_TopMnt_Horizontal
- R3, R4: value 220m 0.5W 1% -> 100m; footprint Resistor_SMD:R_0805_2012Metric -> Resistor_SMD:R_0603_1608Metric
- R5: value 20k -> 23k
- U1: footprint DRV8825_local:PWP28_TI_1p5x0p45_EP3p1x5p18 -> DRV8825:PWP28_5P18X3P1
- U11, U2: value DRV8874PWPR -> a
- U12: value LM7805MP/NOPB -> L7805
- U8: footprint AOZ2261AQI_15:QFN4X4-22L_EP2_S_AOS -> footprints:QFN4X4-22L_EP2_S_AOS
- moved G*** 17.4 mm to (189.3, 88.3)
- moved C31 12.1 mm to (195.8, 86.0), turned to 180 degrees
- moved R5 9.65 mm to (148.9, 91.8), turned to -90 degrees
- moved J3 9.38 mm to (133.8, 114.2), turned to 90 degrees
- moved C30 9.29 mm to (187.0, 91.8), turned to -90 degrees
- moved R24 8.84 mm to (201.2, 97.0), turned to 0 degrees
- moved R23 8.61 mm to (197.8, 97.0), turned to 180 degrees
- moved R6 8.52 mm to (150.4, 91.8), turned to 90 degrees
- moved C34 8.07 mm to (191.4, 95.3)
- moved U8 7.54 mm to (194.8, 91.3)
- moved C32 6.91 mm to (193.0, 95.8)
- moved R25 6.78 mm to (199.2, 94.0), turned to -90 degrees
- moved C2 5.79 mm to (151.4, 88.8), turned to 0 degrees
- moved C3 5.51 mm to (146.8, 97.0), turned to 0 degrees
- moved L1 5.15 mm to (187.5, 82.5), turned to 90 degrees
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Connections:
- J7 pad 12: GPIO4 -> /Microcontroller/GPIO4
- J7 pad 18: GPIO7 -> /Microcontroller/GPIO7
- J7 pad 8: GPIO2 -> /Microcontroller/GPIO2
- U11 pad 17: GND -> (no net)
- U12 pad 4: GND -> (no net)
- U2 pad 17: GND -> (no net)
- U5 pad 10: GPIO7 -> /Microcontroller/GPIO7
- U5 pad 4: GPIO2 -> /Microcontroller/GPIO2
- U5 pad 7: GPIO4 -> /Microcontroller/GPIO4
Routing:
- net GPIO2: track 76.0 -> 0.00 mm, vias 5 -> 0
- net GPIO4: track 72.2 -> 0.00 mm, vias 5 -> 0
- net GPIO7: track 68.4 -> 0.00 mm, vias 5 -> 0
- net GND: track 486.9 -> 546.0 mm, vias 60 -> 29
- net (no net): track 0.00 -> 25.2 mm
- net /Microcontroller/GPIO2: track 0.00 -> 24.9 mm, vias 0 -> 2
- net /Microcontroller/GPIO4: track 0.00 -> 24.2 mm, vias 0 -> 2
- net /Microcontroller/GPIO7: track 0.00 -> 23.2 mm, vias 0 -> 2
- net Net-(C33-Pad2): track 14.8 -> 36.9 mm
- net +12V: track 193.5 -> 209.8 mm, vias 12 -> 13
- net +5V: track 157.6 -> 142.9 mm, vias 8 -> 7
- net Net-(U12-OUT): track 37.0 -> 27.0 mm
- net Net-(U8-BST): track 2.39 -> 11.3 mm, vias 0 -> 2
- net +3V3: track 338.5 -> 329.6 mm, vias 22 -> 24
- net Net-(U1-AVREF): track 11.3 -> 6.11 mm, vias 2 -> 0
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