File: Bucket_universel_v2_before_v2_buck_placement.kicad_pcb (KiCad board)
At the start: 2 copper layers, 100 x 60.5 mm, 128 parts, among them J1 Conn_02x11_Odd_Even, J10 Conn_01x03, J11 Conn_01x03, J12 Conn_01x04_Pin, J13 SM03B-SRSS-TB, J14 Conn_02x18_Odd_Even, J15 USB_C_Receptacle_USB2.0_16P, J2 Conn_01x03_Pin, J3 Conn_01x05_Pin, J4 Conn_01x04_Pin, J5 Conn_01x04_Pin, J7 Conn_02x18_Odd_Even, J8 Conn_01x03, J9 Conn_01x02_Pin, SW1 SW_Push, SW2 SW_Push, U1 DRV8825PWPR, U10 SN74LVC1T45DBV, U11 DRV8874PWPR, U12 LM7805MP/NOPB, U2 DRV8874PWPR, U3 W25Q128JVS, U4 NCP1117-3.3_SOT223, U5 RP2350_60QFN, U7 SN74LVC1T45DBV, U8 AOZ2261AQI-15, U9 SN74LVC1T45DBV, Y1 ABM8-272-T3

Commit message: Yes
Parts:
- J15: footprint Rework_local:USB4105_GND_heel_relief -> Connector_USB:USB_C_Receptacle_GCT_USB4105-xx-A_16P_TopMnt_Horizontal
- R3, R4: value 220m 0.5W 1% -> 100m 0.2W 1%; footprint Resistor_SMD:R_0805_2012Metric -> Resistor_SMD:R_0603_1608Metric
- R5: value 20k -> 56k
- U1: footprint DRV8825_local:PWP28_TI_1p5x0p45_EP3p1x5p18 -> DRV8825_local:PWP28_5P18X3P1_verified
- U11, U2: value DRV8874PWPR -> a
- U12: value LM7805MP/NOPB -> L7805
- moved G*** 17.4 mm to (189.3, 88.3)
- moved R5 9.65 mm to (148.9, 91.8), turned to -90 degrees
- moved R24 8.84 mm to (201.2, 97.0), turned to 0 degrees
- moved C31 8.64 mm to (200.2, 88.9), turned to 90 degrees
- moved R23 8.61 mm to (197.8, 97.0), turned to 180 degrees
- moved R6 8.52 mm to (150.4, 91.8), turned to 90 degrees
- moved U8 7.54 mm to (194.8, 91.3)
- moved C34 7.34 mm to (191.4, 94.6)
- moved R25 7.28 mm to (198.9, 94.4)
- moved C33 7.11 mm to (189.8, 90.6), turned to 90 degrees
- moved C32 6.91 mm to (193.0, 95.8)
- moved C2 5.79 mm to (151.4, 88.8), turned to 0 degrees
- moved C3 5.51 mm to (146.8, 97.0), turned to 0 degrees
- moved R2 4.70 mm to (155.4, 91.2), turned to 90 degrees
- moved R22 4.55 mm to (195.5, 96.2), turned to -90 degrees
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Routing:
- net GND: track 486.9 -> 535.9 mm, vias 60 -> 61
- net +12V: track 193.5 -> 209.0 mm, vias 12 -> 13
- net +3V3: track 338.5 -> 324.0 mm, vias 22 -> 24
- net +5V: track 157.6 -> 146.7 mm, vias 8 -> 7
- net Net-(U12-OUT): track 37.0 -> 26.2 mm
- net Net-(U1-AVREF): track 11.3 -> 6.11 mm, vias 2 -> 0
- net Net-(U1-VCP): track 8.41 -> 4.48 mm
- net Net-(U8-FB): track 3.96 -> 6.95 mm
- net Net-(C33-Pad2): track 14.8 -> 13.2 mm
- net Net-(U2-CPH): track 4.73 -> 3.64 mm
- net Net-(U2-CPL): track 2.91 -> 4.01 mm
- net Net-(U8-BST): track 2.39 -> 3.42 mm
- net Net-(U1-ISENB): track 3.01 -> 2.33 mm
- net Net-(U8-SS): track 3.10 -> 2.43 mm
- net /PSU/Ven: track 11.4 -> 12.0 mm
