File: PSU_before_full_review.kicad_sch (KiCad schematic)
At the start: 21 parts, among them J9 Conn_01x02_Pin, U12 LM7805MP/NOPB, U8 AOZ2261AQI-15

Commit message: Yes
Parts:
- U12: value LM7805MP/NOPB -> L7805; symbol Rework_local:LM7805MP_NOPB_TAB4 -> Regulator_Linear:L7805
- U8: footprint AOZ2261AQI_15:QFN4X4-22L_EP2_S_AOS -> AOZ2261AQI_15:IC_MP2722GRH-0000-Z
Connections:
- net GND: no longer U12.4 (TAB)
Changed lines of the file:
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@@
 	)
 	(symbol
-		(lib_id "Rework_local:LM7805MP_NOPB_TAB4")
+		(lib_id "Regulator_Linear:L7805")
 		(at 153.67 39.37 0)
 		(unit 1)
@@
 			)
 		)
-		(property "Value" "LM7805MP/NOPB"
+		(property "Value" "L7805"
 			(at 153.67 35.56 0)
 			(show_name no)
@@
 			)
 		)
-		(property "Datasheet" "https://www.ti.com/lit/ds/symlink/lm340.pdf"
+		(property "Datasheet" "http://www.st.com/content/ccc/resource/technical/document/datasheet/41/4f/b3/b0/12/d4/47/88/CD00000444.pdf/files/CD00000444.pdf/jcr:content/translations/en.CD00000444.pdf"
 			(at 153.67 40.64 0)
 			(hide yes)
@@
 			)
 		)
-		(property "Description" "TI LM7805MP/NOPB, 5 V linear regulator, SOT-223 DCY, tab pad 4 connected to GND"
+		(property "Description" "Positive 1.5A 35V Linear Regulator, Fixed Output 5V, TO-220/TO-263/TO-252"
 			(at 153.67 39.37 0)
 			(hide yes)
@@
 			)
 		)
-(pin "4")
-)
+	)
 	(symbol
 		(lib_id "power:+5V")
@@
 			)
 		)
-		(property "Footprint" "AOZ2261AQI_15:QFN4X4-22L_EP2_S_AOS"
+		(property "Footprint" "AOZ2261AQI_15:IC_MP2722GRH-0000-Z"
 			(at 140.97 60.706 0)
 			(hide yes)
@@
 		)
 	)
-(wire (pts (xy 153.6700 46.9900) (xy 156.2100 46.9900)) (stroke (width 0) (type default)))
 )
