File: Microcontrolleur.kicad_sch (KiCad schematic)
At the start: 41 parts, among them J13 SM03B-SRSS-TB, J14 Conn_02x18_Odd_Even, J15 USB_C_Receptacle_USB2.0_16P, J7 Conn_02x18_Odd_Even, SW1 SW_Push, SW2 SW_Push, U3 W25Q128JVS, U4 NCP1117-3.3_SOT223, U5 RP2350_60QFN, Y1 ABM8-272-T3

Commit message: V3
Parts:
- removed J13: SM03B-SRSS-TB, Connector_JST:JST_SH_SM03B-SRSS-TB_1x03-1MP_P1.00mm_Horizontal, symbol Connector_Generic_MountingPin:Conn_01x03_MountingPin
- removed J14, J7: Conn_02x18_Odd_Even, Connector_PinHeader_2.54mm:PinHeader_2x18_P2.54mm_Vertical, symbol Connector_Generic:Conn_02x18_Odd_Even
- added H5, H6, H7, H8: MountingHole, MountingHole:MountingHole_2.7mm_M2.5, symbol Mechanical:MountingHole
- J15: footprint Rework_local:USB4105_GND_heel_relief -> Connector_USB:USB_C_Receptacle_GCT_USB4105-xx-A_16P_TopMnt_Horizontal
- R13, R15: now fitted
Connections:
- net GPIO26_ADC0 renamed GPIO26
- net GPIO27_ADC1 renamed GPIO27
- net GPIO28_ADC2 renamed GPIO28
- net GPIO29_ADC3 renamed GPIO29
Other:
- note removed: "IOs"
- note removed: "JST Debug Connector"
