File: backups/drc_cleanup_2026-09-07/Bucket_universel_v2.kicad_pcb (KiCad board)
At the start: 2 copper layers, 100 x 60.5 mm, 128 parts, among them J1 Conn_02x11_Odd_Even, J10 Conn_01x03, J11 Conn_01x03, J12 Conn_01x04_Pin, J13 SM03B-SRSS-TB, J14 Conn_02x18_Odd_Even, J15 USB_C_Receptacle_USB2.0_16P, J2 Conn_01x03_Pin, J3 Conn_01x05_Pin, J4 Conn_01x04_Pin, J5 Conn_01x04_Pin, J7 Conn_02x18_Odd_Even, J8 Conn_01x03, J9 Conn_01x02_Pin, SW1 SW_Push, SW2 SW_Push, U1 DRV8825PWPR, U10 SN74LVC1T45DBV, U11 DRV8874PWPR, U12 LM7805MP/NOPB, U2 DRV8874PWPR, U3 W25Q128JVS, U4 NCP1117-3.3_SOT223, U5 RP2350_60QFN, U7 SN74LVC1T45DBV, U8 AOZ2261AQI-15, U9 SN74LVC1T45DBV, Y1 ABM8-272-T3

Commit message: Yes
Parts:
- J15: footprint Rework_local:USB4105_GND_heel_relief -> Connector_USB:USB_C_Receptacle_GCT_USB4105-xx-A_16P_TopMnt_Horizontal
- U11, U2: value DRV8874PWPR -> a
- U12: value LM7805MP/NOPB -> L7805
- moved G*** 17.4 mm to (189.3, 88.3)
