File: backups/drc_cleanup_2026-09-07/untitled_before_drv8825_rework.kicad_sch (KiCad schematic)
At the start: 16 parts, among them J3 Conn_01x05_Pin, J4 Conn_01x04_Pin, U1 DRV8825PWPR

Commit message: Yes
Parts:
- R3, R4: value 220m 0.5W 1% -> 100m; footprint Resistor_SMD:R_0805_2012Metric -> Resistor_SMD:R_0603_1608Metric
- R5: value 20k -> 23k
- U1: footprint DRV8825_local:PWP28_TI_1p5x0p45_EP3p1x5p18 -> DRV8825:PWP28_5P18X3P1
Changed lines of the file:
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@@
 			)
 		)
-		(property "Value" "20k"
+		(property "Value" "23k"
 			(at 92.71 144.7799 0)
 			(show_name no)
@@
 			)
 		)
-		(property "Value" "220m 0.5W 1%"
+		(property "Value" "100m"
 			(at 82.55 107.9499 0)
 			(show_name no)
@@
 			)
 		)
-		(property "Footprint" "Resistor_SMD:R_0805_2012Metric"
+		(property "Footprint" "Resistor_SMD:R_0603_1608Metric"
 			(at 78.232 106.68 90)
 			(hide yes)
@@
 			)
 		)
-		(property "Value" "220m 0.5W 1%"
+		(property "Value" "100m"
 			(at 87.63 120.6499 0)
 			(show_name no)
@@
 			)
 		)
-		(property "Footprint" "Resistor_SMD:R_0805_2012Metric"
+		(property "Footprint" "Resistor_SMD:R_0603_1608Metric"
 			(at 83.312 119.38 90)
 			(hide yes)
@@
 			)
 		)
-		(property "Footprint" "DRV8825_local:PWP28_TI_1p5x0p45_EP3p1x5p18"
+		(property "Footprint" "DRV8825:PWP28_5P18X3P1"
 			(at 100.33 88.9 0)
 			(hide yes)
