File: backups/u1_datasheet_rework_2026-09-07/Bucket_universel_v2.kicad_pcb (KiCad board)
At the start: 2 copper layers, 100 x 60.5 mm, 128 parts, among them J1 Conn_02x11_Odd_Even, J10 Conn_01x03, J11 Conn_01x03, J12 Conn_01x04_Pin, J13 SM03B-SRSS-TB, J14 Conn_02x18_Odd_Even, J15 USB_C_Receptacle_USB2.0_16P, J2 Conn_01x03_Pin, J3 Conn_01x05_Pin, J4 Conn_01x04_Pin, J5 Conn_01x04_Pin, J7 Conn_02x18_Odd_Even, J8 Conn_01x03, J9 Conn_01x02_Pin, SW1 SW_Push, SW2 SW_Push, U1 DRV8825PWPR, U10 SN74LVC1T45DBV, U11 DRV8874PWPR, U12 LM7805MP/NOPB, U2 DRV8874PWPR, U3 W25Q128JVS, U4 NCP1117-3.3_SOT223, U5 RP2350_60QFN, U7 SN74LVC1T45DBV, U8 AOZ2261AQI-15, U9 SN74LVC1T45DBV, Y1 ABM8-272-T3

Commit message: Yes
Parts:
- J15: footprint Rework_local:USB4105_GND_heel_relief -> Connector_USB:USB_C_Receptacle_GCT_USB4105-xx-A_16P_TopMnt_Horizontal
- R3, R4: value 220m 0.5W 1% -> 100m 0.2W 1%; footprint Resistor_SMD:R_0805_2012Metric -> Resistor_SMD:R_0603_1608Metric
- R5: value 20k -> 56k
- U1: footprint DRV8825_local:PWP28_TI_1p5x0p45_EP3p1x5p18 -> DRV8825_local:PWP28_5P18X3P1_verified
- U11, U2: value DRV8874PWPR -> a
- U12: value LM7805MP/NOPB -> L7805
- moved G*** 17.4 mm to (189.3, 88.3)
- moved R5 9.65 mm to (148.9, 91.8), turned to -90 degrees
- moved R6 8.52 mm to (150.4, 91.8), turned to 90 degrees
- moved C2 5.79 mm to (151.4, 88.8), turned to 0 degrees
- moved C3 5.51 mm to (146.8, 97.0), turned to 0 degrees
- moved R2 4.70 mm to (155.4, 91.2), turned to 90 degrees
- moved C4 3.17 mm to (156.9, 91.2), turned to 90 degrees
- moved R4 1.05 mm to (152.2, 91.7)
- moved R3 1.01 mm to (153.9, 91.2)
Routing:
- net GND: track 486.9 -> 519.8 mm, vias 60 -> 58
- net +12V: track 193.5 -> 207.9 mm, vias 12 -> 13
- net +3V3: track 338.5 -> 327.1 mm
- net Net-(U1-AVREF): track 11.3 -> 6.11 mm, vias 2 -> 0
- net Net-(U1-VCP): track 8.41 -> 4.48 mm
- net Net-(U1-ISENB): track 3.01 -> 2.33 mm
